Commit message: Modell nicht-rückwärtstreibbares Getriebe, diskrete Aktionen, Δ-Kontakt-Reward
- enforce_non_backdrivable Ratchet pro Substep (env, hand)
- MultiDiscrete Action-Space + diskrete Action-Logik (env, policy_runner)
- potential-inspired Δ-Kontakt-Reward + w_hold (reward, configs)
- Box-Collision für Fingertips (urdf), 10M Steps (ppo.yaml)

File: assets/ar10_description/urdf/ar10.urdf (robot description, URDF)
Before this commit: robot ar10, 35 links, 34 joints
Links:
- link fingertip1: geometry collision box size=.015 .015 .03; visual mesh filename=package://ar10_description/meshes/fingertip-v9.STL scale=.001 .001 .001
- link fingertip2: geometry collision box size=.015 .015 .03; visual mesh filename=package://ar10_description/meshes/fingertip-v9.STL scale=.001 .001 .001
- link fingertip3: geometry collision box size=.015 .015 .03; visual mesh filename=package://ar10_description/meshes/fingertip-v9.STL scale=.001 .001 .001
- link fingertip4: geometry collision box size=.015 .015 .03; visual mesh filename=package://ar10_description/meshes/fingertip-v9.STL scale=.001 .001 .001
- link thumbtip: geometry collision box size=.015 .015 .03; visual mesh filename=package://ar10_description/meshes/fingertip-v9.STL scale=.001 .001 .001
